File: BT_Streamer/BT_Streamer.kicad_pcb (KiCad board)
At the start: 2 copper layers, 30.7 x 45.5 mm, 5 parts, among them J2 +12V_IN, J3 +12V_OUT

Commit message: nesto?!
Routing:
- added copper zone on B.Cu, net GND
